File: fujinet-adam-devkit-mini/fujinet-adam-devkit-mini.kicad_pcb (KiCad board)
At the start: 2 copper layers, 27.9 x 55.3 mm, 38 parts, among them J1 RJ12, P1 ST-TF-003A, Q1 MMBT3904, Q2 MMBT3906, SW1 ButtonA, SW2 ButtonB, SW3 Safe Reset, U1 ESP32-DEVKITC-32U

Commit message: Update docs
Parts:
- U1: value ESP32-DEVKITC-32U -> ESP32-DevKitC-VE
Changed lines of the file:
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@@
   )
   (paper "A4")
+  (title_block
+    (title "FujiNet ADAM Devkit Mini")
+    (date "2023-11-11")
+    (rev "1.0")
+    (company "Chris Tersteeg")
+  )
   (layers
     (0 "F.Cu" signal)
@@
     (fp_arc (start 0.6469 8.64) (mid 2.945408 8.849737) (end 5.168 9.472)
       (stroke (width 0.127) (type solid)) (layer "F.SilkS"))
-    (fp_arc (start 6.1679 9.656) (mid 5.659554 9.609621) (end 5.168 9.472)
+    (fp_arc (start 6.1679 9.656) (mid 5.659557 9.609613) (end 5.168 9.472)
       (stroke (width 0.127) (type solid)) (layer "F.SilkS"))
     (fp_poly
@@
         (effects (font (size 1 1) (thickness 0.015)) (justify mirror))
     )
-    (fp_text value "ESP32-DEVKITC-32U" (at 1.27 -26.035) (layer "B.Fab")
-        (effects (font (size 1 1) (thickness 0.015)) (justify mirror))
+    (fp_text value "ESP32-DevKitC-VE" (at 0 -21.854) (layer "B.SilkS")
+        (effects (font (size 1 1) (thickness 0.15)) (justify mirror))
     )
     (fp_line (start -13.95 -24.1) (end -4.07 -24.1)
