File: fujinet-adam-devkit-mini/fujinet-adam-devkit-mini.kicad_sch (KiCad schematic)
At the start: 38 parts, among them J1 RJ12, P1 ST-TF-003A, Q1 MMBT3904, Q2 MMBT3906, SW1 ButtonA, SW2 ButtonB, SW3 Safe Reset, U1 ESP32-DEVKITC-32U

Commit message: Update docs
Parts:
- U1: value ESP32-DEVKITC-32U -> ESP32-DevKitC-VE
Changed lines of the file:
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@@
       (effects (font (size 1.27 1.27)))
     )
-    (property "Value" "ESP32-DEVKITC-32U" (at 189.23 37.465 0)
+    (property "Value" "ESP32-DevKitC-VE" (at 189.23 37.465 0)
       (effects (font (size 1.27 1.27)))
     )
