File: fujinet-adam-devkit-smd/fujinet-adam-devkit-smd.kicad_sch (KiCad schematic)
At the start: 39 parts, among them J1 RJ12, J2 RJ12, J3 SD_Card, Q1 MMBT3904, Q2 MMBT3906, SW1 ButtonA, SW2 ButtonB, SW3 Safe Reset, U1 ESP32-DEVKITC-32U

Commit message: Update docs
Parts:
- U1: value ESP32-DEVKITC-32U -> ESP32-DevKitC-VE
Other:
- title: Fujinet ADAM DevKit Mini -> Fujinet ADAM DevKit SMD

Commit message: Update SMD PCB and Case to v1.1, fix ADAMNet Out port not working
Parts:
- J1: value RJ12 -> In
- J2: value RJ12 -> Out
Connections:
- net ADAMNET_5V: now also J2.1; no longer J2.6
- net ADAMNET_DATA: now also J2.6; no longer J2.1
- net ADAMNET_RESET: now also J2.5; no longer J2.2
- net GND: now also J2.2; no longer J2.5
Changed lines of the file:
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@@
   (title_block
     (title "Fujinet ADAM DevKit SMD")
-    (date "2023-11-11")
-    (rev "1.0")
+    (date "2023-12-25")
+    (rev "1.1")
     (company "Chris Tersteeg")
   )
@@
   (junction (at 43.815 88.265) (diameter 0) (color 0 0 0 0)
   )
-  (junction (at 88.265 89.535) (diameter 0) (color 0 0 0 0)
-  )
   (junction (at 69.85 149.86) (diameter 0) (color 0 0 0 0)
   )
@@
   (junction (at 102.235 160.655) (diameter 0) (color 0 0 0 0)
   )
+  (junction (at 87.122 84.582) (diameter 0) (color 0 0 0 0)
+  )
   (junction (at 150.495 164.465) (diameter 0) (color 0 0 0 0)
   )
@@
   (junction (at 73.66 122.555) (diameter 0) (color 0 0 0 0)
   )
+  (junction (at 87.122 82.042) (diameter 0) (color 0 0 0 0)
+  )
   (junction (at 238.125 151.765) (diameter 0) (color 0 0 0 0)
   )
@@
   )
   (junction (at 54.61 122.555) (diameter 0) (color 0 0 0 0)
-  )
-  (junction (at 88.265 86.995) (diameter 0) (color 0 0 0 0)
   )
   (junction (at 69.85 122.555) (diameter 0) (color 0 0 0 0)
@@
     (stroke (width 0) (type default))
   )
-  (wire (pts (xy 85.09 92.075) (xy 98.425 92.075))
+  (wire (pts (xy 85.09 84.582) (xy 87.122 84.582))
     (stroke (width 0) (type default))
   )
@@
     (stroke (width 0) (type default))
   )
+  (wire (pts (xy 85.09 87.122) (xy 87.122 87.122))
+    (stroke (width 0) (type default))
+  )
   (wire (pts (xy 209.55 42.545) (xy 233.68 42.545))
     (stroke (width 0) (type default))
@@
     (stroke (width 0) (type default))
   )
-  (wire (pts (xy 85.09 81.915) (xy 101.6 81.915))
-    (stroke (width 0) (type default))
-  )
   (wire (pts (xy 80.645 117.475) (xy 80.645 122.555))
     (stroke (width 0) (type default))
@@
     (stroke (width 0) (type default))
   )
-  (wire (pts (xy 88.265 89.535) (xy 85.09 89.535))
-    (stroke (width 0) (type default))
-  )
   (wire (pts (xy 209.55 60.325) (xy 227.33 60.325))
     (stroke (width 0) (type default))
@@
     (stroke (width 0) (type default))
   )
-  (wire (pts (xy 88.265 89.535) (xy 102.235 89.535))
-    (stroke (width 0) (type default))
-  )
   (wire (pts (xy 163.83 135.89) (xy 165.735 135.89))
     (stroke (width 0) (type default))
   )
+  (wire (pts (xy 101.092 89.662) (xy 85.09 89.662))
+    (stroke (width 0) (type default))
+  )
   (wire (pts (xy 250.19 151.765) (xy 252.095 151.765))
     (stroke (width 0) (type default))
@@
     (stroke (width 0) (type default))
   )
+  (wire (pts (xy 87.122 84.582) (xy 87.122 87.122))
+    (stroke (width 0) (type default))
+  )
   (wire (pts (xy 227.33 151.765) (xy 238.125 151.765))
     (stroke (width 0) (type default))
   )
-  (wire (pts (xy 88.265 84.455) (xy 88.265 86.995))
-    (stroke (width 0) (type default))
-  )
   (wire (pts (xy 54.61 152.4) (xy 77.47 152.4))
     (stroke (width 0) (type default))
@@
     (stroke (width 0) (type default))
   )
+  (wire (pts (xy 87.122 82.042) (xy 87.122 84.582))
+    (stroke (width 0) (type default))
+  )
   (wire (pts (xy 238.125 97.79) (xy 238.125 101.6))
     (stroke (width 0) (type default))
@@
     (stroke (width 0) (type default))
   )
-  (wire (pts (xy 85.09 79.375) (xy 100.33 79.375))
-    (stroke (width 0) (type default))
-  )
   (wire (pts (xy 173.355 123.825) (xy 173.355 130.81))
     (stroke (width 0) (type default))
@@
     (stroke (width 0) (type default))
   )
+  (wire (pts (xy 101.092 92.202) (xy 85.09 92.202))
+    (stroke (width 0) (type default))
+  )
   (wire (pts (xy 43.815 85.725) (xy 40.64 85.725))
     (stroke (width 0) (type default))
@@
     (stroke (width 0) (type default))
   )
-  (wire (pts (xy 88.265 86.995) (xy 85.09 86.995))
-    (stroke (width 0) (type default))
-  )
   (wire (pts (xy 238.125 151.765) (xy 240.03 151.765))
     (stroke (width 0) (type default))
@@
     (stroke (width 0) (type default))
   )
-  (wire (pts (xy 88.265 86.995) (xy 88.265 89.535))
-    (stroke (width 0) (type default))
-  )
   (wire (pts (xy 147.955 75.565) (xy 147.955 78.74))
     (stroke (width 0) (type default))
@@
     (stroke (width 0) (type default))
   )
+  (wire (pts (xy 104.394 82.042) (xy 87.122 82.042))
+    (stroke (width 0) (type default))
+  )
   (wire (pts (xy 191.135 116.205) (xy 207.01 116.205))
     (stroke (width 0) (type default))
@@
     (stroke (width 0) (type default))
   )
+  (wire (pts (xy 87.122 82.042) (xy 85.09 82.042))
+    (stroke (width 0) (type default))
+  )
   (wire (pts (xy 69.85 142.24) (xy 69.85 149.86))
     (stroke (width 0) (type default))
@@
     (stroke (width 0) (type default))
   )
+  (wire (pts (xy 100.838 79.502) (xy 85.09 79.502))
+    (stroke (width 0) (type default))
+  )
   (wire (pts (xy 43.815 90.805) (xy 57.785 90.805))
-    (stroke (width 0) (type default))
-  )
-  (wire (pts (xy 88.265 84.455) (xy 85.09 84.455))
     (stroke (width 0) (type default))
   )
@@
     (effects (font (size 1.27 1.27)) (justify left bottom))
   )
-  (label "ADAMNET_RESET" (at 101.6 81.915 180) (fields_autoplaced)
+  (label "ADAMNET_RESET" (at 101.092 89.662 180) (fields_autoplaced)
     (effects (font (size 1.27 1.27)) (justify right bottom))
   )
@@
     (effects (font (size 1.27 1.27)) (justify right bottom))
   )
-  (label "ADAMNET_5V" (at 98.425 92.075 180) (fields_autoplaced)
+  (label "ADAMNET_5V" (at 100.838 79.502 180) (fields_autoplaced)
     (effects (font (size 1.27 1.27)) (justify right bottom))
   )
@@
     (effects (font (size 1.27 1.27)) (justify right bottom))
   )
-  (label "ADAMNET_DATA" (at 100.33 79.375 180) (fields_autoplaced)
+  (label "ADAMNET_DATA" (at 101.092 92.202 180) (fields_autoplaced)
     (effects (font (size 1.27 1.27)) (justify right bottom))
   )
@@
       (effects (font (size 1.27 1.27)))
     )
-    (property "Value" "RJ12" (at 30.48 97.79 0)
+    (property "Value" "In" (at 30.48 97.79 0)
       (effects (font (size 1.27 1.27)))
     )
@@
     )
   )
-  (symbol (lib_id "power:GND") (at 102.235 89.535 0) (unit 1)
-    (in_bom yes) (on_board yes) (dnp no) (fields_autoplaced)
-    (property "Reference" "#PWR025" (at 102.235 95.885 0)
-      (effects (font (size 1.27 1.27)) hide)
-    )
-    (property "Value" "GND" (at 102.235 94.615 0)
-      (effects (font (size 1.27 1.27)))
-    )
-    (property "Footprint" "" (at 102.235 89.535 0)
-      (effects (font (size 1.27 1.27)) hide)
-    )
-    (property "Datasheet" "" (at 102.235 89.535 0)
+  (symbol (lib_id "power:GND") (at 104.394 82.042 0) (unit 1)
+    (in_bom yes) (on_board yes) (dnp no) (fields_autoplaced)
+    (property "Reference" "#PWR025" (at 104.394 88.392 0)
+      (effects (font (size 1.27 1.27)) hide)
+    )
+    (property "Value" "GND" (at 104.394 87.122 0)
+      (effects (font (size 1.27 1.27)))
+    )
+    (property "Footprint" "" (at 104.394 82.042 0)
+      (effects (font (size 1.27 1.27)) hide)
+    )
+    (property "Datasheet" "" (at 104.394 82.042 0)
       (effects (font (size 1.27 1.27)) hide)
     )
@@
     )
   )
-  (symbol (lib_id "Connector:RJ12") (at 74.93 84.455 0) (mirror x) (unit 1)
+  (symbol (lib_id "Connector:RJ12") (at 74.93 84.582 0) (mirror x) (unit 1)
     (in_bom yes) (on_board yes) (dnp no)
-    (property "Reference" "J2" (at 74.93 99.06 0)
-      (effects (font (size 1.27 1.27)))
-    )
-    (property "Value" "RJ12" (at 74.93 96.52 0)
-      (effects (font (size 1.27 1.27)))
-    )
-    (property "Footprint" "Connector_RJ:RJ12_Amphenol_54601" (at 74.93 85.09 90)
-      (effects (font (size 1.27 1.27)) hide)
-    )
-    (property "Datasheet" "~" (at 74.93 85.09 90)
-      (effects (font (size 1.27 1.27)) hide)
-    )
+    (property "Reference" "J2" (at 74.93 99.187 0)
+      (effects (font (size 1.27 1.27)))
+    )
+    (property "Value" "Out" (at 74.93 96.647 0)
+      (effects (font (size 1.27 1.27)))
+    )
+    (property "Footprint" "Connector_RJ:RJ12_Amphenol_54601" (at 74.93 85.217 90)
+      (effects (font (size 1.27 1.27)) hide)
+    )
+    (property "Datasheet" "~" (at 74.93 85.217 90)
+      (effects (font (size 1.27 1.27)) hide)
+    )

Commit message: Add SMD version 1.2 PCB/case files and embossed text STL's for AMS printing
Parts:
- added JP1: Always On, Jumper:SolderJumper-2_P1.3mm_Open_RoundedPad1.0x1.5mm, symbol Jumper:SolderJumper_2_Open
- added S1: SK12D07VG4, SK12D07VG4:SK12D07VG4, symbol SK12D07VG4:SK12D07VG4
Connections:
- net ADAMNET_5V: now also JP1.1 (A), S1.COM; no longer D4.2 (A)
- new net: D4.2 (A), JP1.2 (B), S1.1
- no-connect marks 19 -> 20
Other:
- moved on the sheet: C2, D4
